File: TivaClock.sch (KiCad schematic (older format))
At the start: 7 parts, among them J1 Conn_01x10, J2 Conn_01x10, J3 Conn_01x10, J4 Conn_01x10, J5 Conn_01x20, J6 Conn_01x20, J7 GS3

Commit message: Add pin names to launchpad headers
Other:
- note added: "3.3V\nPB5\nPB0\nPB1\nPE4\nPE5\nPB4\nPA5\nPA6\nPA7"
- note added: "GND\nPB2\nPE0\nPF0\nRST\nPB7\nPB6\nPA4\nPA3\nPA2"
- note added: "PF2\nPF3\nPB3\nPC4\nPC5\nPC6\nPC7\nPD6\nPD7\nPF4"
- note added: "VBUS\nGND\nPD0\nPD1\nPD2\nPD3\nPE1\nPE2\nPE3\nPF1"
Changed lines of the file:
@@
 NoConn ~ 5000 5350
 NoConn ~ 5000 5450
+Text Notes 2850 2850 0    63   ~ 0
+3.3V\nPB5\nPB0\nPB1\nPE4\nPE5\nPB4\nPA5\nPA6\nPA7
+Text Notes 3100 2850 0    63   ~ 0
+VBUS\nGND\nPD0\nPD1\nPD2\nPD3\nPE1\nPE2\nPE3\nPF1
+Text Notes 7850 2850 0    63   ~ 0
+PF2\nPF3\nPB3\nPC4\nPC5\nPC6\nPC7\nPD6\nPD7\nPF4
+Text Notes 8250 2850 0    63   ~ 0
+GND\nPB2\nPE0\nPF0\nRST\nPB7\nPB6\nPA4\nPA3\nPA2
 $EndSCHEMATC
